File: Hardware/0. Project/PartsHunter Slave/PartsHunter Slave.brd (EAGLE design)
At the start: 210 x 150 mm, 37 parts, among them IC1 PCF8574P

Commit message: rearranged components positions at PCB layout
Parts:
- moved R7 174.7 mm to (116.0, 64.6), turned to 180 degrees
- moved R3 170.4 mm to (98.0, 64.6)
- moved R5 165.7 mm to (116.0, 69.7), turned to 180 degrees
- moved R2 161.8 mm to (116.0, 74.8)
- moved R8 156.1 mm to (116.0, 77.3)
- moved R1 155.5 mm to (116.0, 72.2), turned to 0 degrees
- moved R4 154.1 mm to (98.0, 67.2), turned to 180 degrees
- moved R9 150.4 mm to (116.0, 79.8)
- moved R6 150.1 mm to (116.0, 67.2)
- moved SW1 36.0 mm to (107.0, 38.0)
- moved LED1 22.5 mm to (185.0, 126.0)
- moved LED5 20.8 mm to (185.0, 91.0)
- moved LED13 20.0 mm to (185.0, 21.0)
- moved LED9 19.9 mm to (185.0, 56.0)
- moved JP3 19.2 mm to (159.0, 1.00)
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Other:
- board size 210 x 150 mm -> 214 x 147 mm
